File: 514_final/schematic/schematic.kicad_pcb (KiCad board)
At the start: 2 copper layers, 62.5 x 45 mm, 18 parts, among them M1 Stepper_Motor_bipolar, SW1 SW_SPST, SW2 SW_SPST

Commit message: 0301
Parts:
- removed BH1750: light sensor, Connector_PinHeader_2.54mm:PinHeader_1x04_P2.54mm_Vertical
- removed C1: 0.1μF, Capacitor_SMD:C_0805_2012Metric
- removed C3: 10μF, Capacitor_SMD:C_0805_2012Metric
- removed D1: LED, LED_SMD:LED_0805_2012Metric
- removed DFRobot_SEN0161-V2: pH sensor, Connector_PinHeader_2.54mm:PinHeader_1x03_P2.54mm_Vertical
- removed DFRobot_SEN0193: moisture sensor, Connector_PinHeader_2.54mm:PinHeader_1x03_P2.54mm_Vertical
- removed R1, R2: 4.7kΩ, Capacitor_SMD:C_0805_2012Metric
- removed R3: 330Ω, Capacitor_SMD:C_0805_2012Metric
- removed SW1: SW_SPST, Button_Switch_THT:SW_PUSH_6mm
- removed U1: ~, 514final_Library:XIAO_ESP32
- added REF**: MountingHole_2.7mm, MountingHole:MountingHole_2.7mm, F.Cu at (210.0, 82.5)
- added REF**: MountingHole_2.7mm, MountingHole:MountingHole_2.7mm, F.Cu at (157.5, 117.5)
