File: 514_final/schematic - 0222/schematic.kicad_pcb (KiCad board)
At the start: 2 copper layers, 62.5 x 45 mm, 9 parts, among them M1 Stepper_Motor_bipolar, SW2 SW_SPST

Commit message: final
Routing:
- net Net-(D2-A): track 0.00 -> 6.61 mm
Changed lines of the file:
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@@
+	)
+	(segment
+		(start 208.4375 100)
+		(end 207.4365 98.999)
+		(width 0.2)
+		(layer "F.Cu")
+		(net 15)
+	)
+	(segment
+		(start 203.541 98.999)
+		(end 202.62 99.92)
+		(width 0.2)
+		(layer "F.Cu")
+		(net 15)
+	)
+	(segment
+		(start 207.4365 98.999)
+		(end 203.541 98.999)
+		(width 0.2)
+		(layer "F.Cu")
+		(net 15)
 	)
 	(segment
